Commit message: just change the color of the inmoov face

File: ros/kit_head/kit_head_description/model/kit_head.urdf.xacro (robot description, xacro)
@@ -220,5 +220,5 @@
           <mesh filename="package://kit_head_description/meshes/inmoov_face.stl"/>
         </geometry>
-        <material name="KIT/White"/>
+        <material name="KIT/Orange"/>
       </visual>
       <collision>

Commit message: removing the inmoov face

File: ros/kit_head/kit_head_description/model/kit_head.urdf.xacro (robot description, xacro)
@@ -209,5 +209,5 @@
       </collision>
     </link>
-    <joint name="${name}_face_joint" type="fixed">
+<!--     <joint name="${name}_face_joint" type="fixed">
       <origin xyz="0.05 -0.02 0" rpy="-1.57 2.356194 0.0" />
       <parent link="${name}_head_5_link"/>
@@ -228,5 +228,5 @@
         </geometry>
       </collision>
-    </link>
+    </link> -->
   </xacro:macro>
 </robot>

Commit message: update with kinect and camera simulation support

File: ros/kit_head/kit_head_description/model/kit_head.urdf.xacro (robot description, xacro)
@@ -2,4 +2,7 @@
 <robot xmlns:xacro="http://www.ros.org/wiki/xacro">
   <xacro:include filename="$(find kit_head_description)/model/materials.urdf"/>
+  <xacro:include filename="$(find kit_head_description)/model/kit_head.inertia.xacro"/>
+  <xacro:include filename="$(find kit_head_description)/model/kit_head.transmission.xacro"/>
+  <xacro:include filename="$(find kit_head_description)/model/kit_head.gazebo.xacro"/>
   <xacro:property name="M_PI" value="3.1415926535897931" />
   <xacro:property name="velocity_scale_factor" value="1.0"/>
@@ -9,7 +12,24 @@
       <insert_block name="origin"/>
       <parent link="${parent}"/>
-      <child link="calib_${name}_base_link"/>
-    </joint>
-    <link name="calib_${name}_base_link" />
+      <child link="${name}_base_link"/>
+    </joint>
+    <link name="${name}_base_link">
+      <inertial>
+        <insert_block name="negligible_inertia"/>
+      </inertial>
+      <!-- <visual>
+        <origin xyz="0 0 0" rpy="0 0 0"/>
+        <geometry>
+          <cylinder radius="0.03" length="0.15"/>
+        </geometry>
+        <material name="KIT/DarkGrey"/>
+      </visual>
+      <collision>
+        <origin xyz="0 0 0" rpy="0 0 0"/>
+        <geometry>
+          <cylinder radius="0.03" length="0.15"/>
+        </geometry>
+      </collision> -->
+    </link>
     <!-- neck -->
     <joint name="${name}_neck_pitch_joint" type="revolute">
@@ -22,9 +42,12 @@
                          k_position="30"
                          k_velocity="30"/>
-      <dynamics damping="1.0"/>
-      <parent link="calib_${name}_base_link"/>
+      <dynamics friction="1.0" damping="1.0"/>
+      <parent link="${name}_base_link"/>
       <child link="${name}_head_1_link"/>
     </joint>
     <link name="${name}_head_1_link">
+      <inertial>
+        <insert_block name="negligible_inertia"/>
+      </inertial>
       <visual>
         <origin xyz="0 0 0" rpy="0 0 0"/>
@@ -50,9 +73,12 @@
                          k_position="30"
                          k_velocity="30"/>
-      <dynamics damping="1.0"/>
+      <dynamics friction="1.0" damping="1.0"/>
       <parent link="${name}_head_1_link"/>
       <child link="${name}_head_2_link"/>
     </joint>
     <link name="${name}_head_2_link">
+      <inertial>
+        <insert_block name="negligible_inertia"/>
+      </inertial>
       <visual>
         <origin xyz="0 0 0" rpy="0 0 0"/>
@@ -78,9 +104,12 @@
                          k_position="30"
                          k_velocity="30"/>
-      <dynamics damping="1.0"/>
+      <dynamics friction="1.0" damping="1.0"/>
       <parent link="${name}_head_2_link"/>
       <child link="${name}_head_3_link"/>
     </joint>
     <link name="${name}_head_3_link">
+      <inertial>
+        <insert_block name="negligible_inertia"/>
+      </inertial>
       <visual>
         <origin xyz="0 0 0" rpy="0 0 0"/>
@@ -106,9 +135,12 @@
                          k_position="30"
                          k_velocity="30"/>
-      <dynamics damping="1.0"/>
+      <dynamics friction="1.0" damping="1.0"/>
       <parent link="${name}_head_3_link"/>
       <child link="${name}_head_4_link"/>
     </joint>
     <link name="${name}_head_4_link">
+      <inertial>
+        <insert_block name="negligible_inertia"/>
+      </inertial>
       <visual>
         <origin xyz="0 0 0" rpy="0 0 0"/>
@@ -134,9 +166,12 @@
                          k_position="30"
                          k_velocity="30"/>
-      <dynamics damping="1.0"/>
+      <dynamics friction="1.0" damping="1.0"/>
       <parent link="${name}_head_4_link"/>
       <child link="${name}_head_5_link"/>
     </joint>
     <link name="${name}_head_5_link">
+      <inertial>
+        <insert_block name="negligible_inertia"/>
+      </inertial>
       <visual>
         <origin xyz="0 0 0" rpy="0 0 0"/>
@@ -162,9 +197,12 @@
                          k_position="30"
                          k_velocity="30"/>
-      <dynamics damping="1.0"/>
+      <dynamics friction="1.0" damping="1.0"/>
       <parent link="${name}_head_5_link"/>
       <child link="${name}_left_eye_link"/>
     </joint>
     <link name="${name}_left_eye_link">
+      <inertial>
+        <insert_block name="negligible_inertia"/>
+      </inertial>
       <visual>
         <origin xyz="0.02 0 0" rpy="0 ${M_PI/2} 0"/>
@@ -190,9 +228,12 @@
                          k_position="30"
                          k_velocity="30"/>
-      <dynamics damping="1.0"/>
+      <dynamics friction="1.0" damping="1.0"/>
       <parent link="${name}_head_5_link"/>
       <child link="${name}_right_eye_link"/>
     </joint>
     <link name="${name}_right_eye_link">
+      <inertial>
+        <insert_block name="negligible_inertia"/>
+      </inertial>
       <visual>
         <origin xyz="0.02 0 0" rpy="0 ${M_PI/2} 0"/>
@@ -229,4 +270,29 @@
       </collision>
     </link> -->
+    <joint name="${name}_asus_joint" type="fixed">
+      <origin xyz="0 -0.1 0" rpy="1.5707 0.0 0.0"/>
+      <parent link="${name}_head_5_link"/>
+      <child link="${name}_asus_link"/>
+    </joint>
+    <link name="${name}_asus_link">
+      <inertial>
+        <insert_block name="negligible_inertia"/>
+      </inertial>
+      <visual>
+        <origin xyz="0 0 0" rpy="0 0 0"/>
+        <geometry>
+          <mesh filename="package://kit_head_description/meshes/asus_xtion_body.stl"/>
+        </geometry>
+        <material name="KIT/Black"/>
+      </visual>
+      <collision>
+        <origin xyz="0 0 0" rpy="0 0 0"/>
+        <geometry>
+          <cylinder radius="0.03" length="0.15"/>
+        </geometry>
+      </collision>
+    </link>
+    <xacro:kit_head_transmission name="${name}"/>
+    <xacro:kit_head_gazebo name="${name}"/>
   </xacro:macro>
 </robot>
