Commit message: Updated collision geometry

File: kit_head_description/model/kit_head.urdf.xacro (robot description, xacro)
@@ -182,7 +182,7 @@
       </visual>
       <collision>
-        <origin xyz="0 0.18 0" rpy="${M_PI/2} 0 0"/>
-        <geometry>
-          <cylinder radius="0.15" length="0.4"/>s
+        <origin xyz="-0.1 0.10 0" rpy="${M_PI/2} 0 0"/>
+        <geometry>
+          <cylinder radius="0.12" length="0.3"/>
         </geometry>
       </collision>
@@ -213,5 +213,5 @@
       </visual>
       <collision>
-        <origin xyz="0.02 0 0" rpy="0 0 0"/>
+        <origin xyz="0.02 0 0" rpy="0 ${M_PI/2} 0"/>
         <geometry>
           <cylinder radius="0.03" length="0.02"/>
@@ -244,5 +244,5 @@
       </visual>
       <collision>
-        <origin xyz="0.02 0 0" rpy="0 0 0"/>
+        <origin xyz="0.02 0 0" rpy="0 ${M_PI/2} 0"/>
         <geometry>
           <cylinder radius="0.03" length="0.02"/>
@@ -287,7 +287,7 @@
       </visual>
       <collision>
-        <origin xyz="0 0 0" rpy="0 0 0"/>
-        <geometry>
-          <cylinder radius="0.03" length="0.15"/>
+        <origin xyz="0 0 0" rpy="${M_PI/2} 0 0"/>
+        <geometry>
+          <cylinder radius="0.03" length="0.20"/>
         </geometry>
       </collision>

Commit message: Corrected the kinematics in the urdf according to our head, added individual eyes as well and renamed links to more descriptive names

File: kit_head_description/model/kit_head.urdf.xacro (robot description, xacro)
@@ -44,7 +44,7 @@
       <dynamics friction="1.0" damping="1.0"/>
       <parent link="${name}_base_link"/>
-      <child link="${name}_head_1_link"/>
-    </joint>
-    <link name="${name}_head_1_link">
+      <child link="${name}_neck_pitch_link"/>
+    </joint>
+    <link name="${name}_neck_pitch_link">
       <inertial>
         <xacro:insert_block name="negligible_inertia"/>
@@ -74,8 +74,8 @@
                          k_velocity="30"/>
       <dynamics friction="1.0" damping="1.0"/>
-      <parent link="${name}_head_1_link"/>
-      <child link="${name}_head_2_link"/>
-    </joint>
-    <link name="${name}_head_2_link">
+      <parent link="${name}_neck_pitch_link"/>
+      <child link="${name}_neck_roll_link"/>
+    </joint>
+    <link name="${name}_neck_roll_link">
       <inertial>
         <xacro:insert_block name="negligible_inertia"/>
@@ -105,27 +105,27 @@
                          k_velocity="30"/>
       <dynamics friction="1.0" damping="1.0"/>
-      <parent link="${name}_head_2_link"/>
-      <child link="${name}_head_3_link"/>
-    </joint>
-    <link name="${name}_head_3_link">
-      <inertial>
-        <xacro:insert_block name="negligible_inertia"/>
-      </inertial>
-      <visual>
-        <origin xyz="0 0 0" rpy="0 0 0"/>
-        <geometry>
-          <cylinder radius="0.03" length="0.15"/>
-        </geometry>
-        <material name="KIT/DarkGrey"/>
-      </visual>
-      <collision>
-        <origin xyz="0 0 0" rpy="0 0 0"/>
-        <geometry>
-          <cylinder radius="0.03" length="0.15"/>
-        </geometry>
-      </collision>
-    </link>
-    <joint name="${name}_head_tilt_joint" type="revolute">
-      <origin xyz="0 0 -0.1745" rpy="${M_PI/2} 0 0"/>
+      <parent link="${name}_neck_roll_link"/>
+      <child link="${name}_neck_yaw_link"/>
+    </joint>
+    <link name="${name}_neck_yaw_link">
+      <inertial>
+        <xacro:insert_block name="negligible_inertia"/>
+      </inertial>
+      <visual>
+        <origin xyz="0 0 0" rpy="0 0 0"/>
+        <geometry>
+          <cylinder radius="0.03" length="0.15"/>
+        </geometry>
+        <material name="KIT/DarkGrey"/>
+      </visual>
+      <collision>
+        <origin xyz="0 0 0" rpy="0 0 0"/>
+        <geometry>
+          <cylinder radius="0.03" length="0.15"/>
+        </geometry>
+      </collision>
+    </link>
+    <joint name="${name}_neck_tilt_joint" type="revolute">
+      <origin xyz="0 0 -0.122" rpy="${M_PI/2} 0 0"/>
       <axis xyz="0 0 1"/>
       <limit lower="${-40 * M_PI / 180}" upper="${40 * M_PI / 180}"
@@ -136,8 +136,8 @@
                          k_velocity="30"/>
       <dynamics friction="1.0" damping="1.0"/>
-      <parent link="${name}_head_3_link"/>
-      <child link="${name}_head_4_link"/>
-    </joint>
-    <link name="${name}_head_4_link">
+      <parent link="${name}_neck_yaw_link"/>
+      <child link="${name}_neck_tilt_link"/>
+    </joint>
+    <link name="${name}_neck_tilt_link">
       <inertial>
         <xacro:insert_block name="negligible_inertia"/>
@@ -158,5 +158,5 @@
     </link>
     <joint name="${name}_eyes_tilt_joint" type="revolute">
-      <origin xyz="0.1 0 0" rpy="0 0 0"/>
+      <origin xyz="0.1 -0.0525 0.0" rpy="0 0 0"/>
       <axis xyz="0 0 1"/>
       <limit lower="${-20 * M_PI / 180}" upper="${20 * M_PI / 180}"
@@ -167,8 +167,8 @@
                          k_velocity="30"/>
       <dynamics friction="1.0" damping="1.0"/>
-      <parent link="${name}_head_4_link"/>
-      <child link="${name}_head_5_link"/>
-    </joint>
-    <link name="${name}_head_5_link">
+      <parent link="${name}_neck_tilt_link"/>
+      <child link="${name}_eyes_tilt_link"/>
+    </joint>
+    <link name="${name}_eyes_tilt_link">
       <inertial>
         <xacro:insert_block name="negligible_inertia"/>
@@ -198,22 +198,45 @@
                          k_velocity="30"/>
       <dynamics friction="1.0" damping="1.0"/>
-      <parent link="${name}_head_5_link"/>
-      <child link="${name}_left_eye_link"/>
-    </joint>
-    <link name="${name}_left_eye_link">
-      <inertial>
-        <xacro:insert_block name="negligible_inertia"/>
-      </inertial>
-      <visual>
-        <origin xyz="0.02 0 0" rpy="0 ${M_PI/2} 0"/>
-        <geometry>
-          <cylinder radius="0.03" length="0.02"/>
+      <parent link="${name}_eyes_tilt_link"/>
+      <child link="${name}_left_eye_peripheral_link"/>
+    </joint>
+    <link name="${name}_left_eye_peripheral_link">
+      <inertial>
+        <xacro:insert_block name="negligible_inertia"/>
+      </inertial>
+      <visual>
+        <origin xyz="0.0 0 0.018" rpy="0 ${M_PI/2} 0"/>
+        <geometry>
+          <sphere radius="0.018"/>
         </geometry>
         <material name="KIT/White"/>
       </visual>
       <collision>
-        <origin xyz="0.02 0 0" rpy="0 ${M_PI/2} 0"/>
-        <geometry>
-          <cylinder radius="0.03" length="0.02"/>
+        <origin xyz="0.0 0 0" rpy="0 ${M_PI/2} 0"/>
+        <geometry>
+          <sphere radius="0.018"/>
+        </geometry>
+      </collision>
+    </link>
+    <joint name="${name}_left_eye_foveal_joint" type="fixed">
+      <origin xyz="0 0 -0.018" rpy="0.0 0.0 0.0"/>
+      <parent link="${name}_left_eye_peripheral_link"/>
+      <child link="${name}_left_eye_foveal_link"/>
+    </joint>
+    <link name="${name}_left_eye_foveal_link">
+      <inertial>
+        <xacro:insert_block name="negligible_inertia"/>
+      </inertial>
+      <visual>
+        <origin xyz="0 0 0" rpy="0 0 0"/>
+        <geometry>
+          <sphere radius="0.018"/>
+        </geometry>
+        <material name="KIT/White"/>
+      </visual>
+      <collision>
+        <origin xyz="0 0 0" rpy="0 0 0"/>
+        <geometry>
+          <sphere radius="0.018"/>
         </geometry>
       </collision>
@@ -229,22 +252,45 @@
                          k_velocity="30"/>
       <dynamics friction="1.0" damping="1.0"/>
-      <parent link="${name}_head_5_link"/>
-      <child link="${name}_right_eye_link"/>
-    </joint>
-    <link name="${name}_right_eye_link">
-      <inertial>
-        <xacro:insert_block name="negligible_inertia"/>
-      </inertial>
-      <visual>
-        <origin xyz="0.02 0 0" rpy="0 ${M_PI/2} 0"/>
-        <geometry>
-          <cylinder radius="0.03" length="0.02"/>
+      <parent link="${name}_eyes_tilt_link"/>
+      <child link="${name}_right_eye_peripheral_link"/>
+    </joint>
+    <link name="${name}_right_eye_peripheral_link">
+      <inertial>
+        <xacro:insert_block name="negligible_inertia"/>
+      </inertial>
+      <visual>
+        <origin xyz="0.0 0 0.018" rpy="0 ${M_PI/2} 0"/>
+        <geometry>
+          <sphere radius="0.018"/>
         </geometry>
         <material name="KIT/White"/>
       </visual>
       <collision>
-        <origin xyz="0.02 0 0" rpy="0 ${M_PI/2} 0"/>
-        <geometry>
-          <cylinder radius="0.03" length="0.02"/>
+        <origin xyz="0.0 0 0" rpy="0 ${M_PI/2} 0"/>
+        <geometry>
+          <sphere radius="0.018"/>
+        </geometry>
+      </collision>
+    </link>
+    <joint name="${name}_right_eye_foveal_joint" type="fixed">
+      <origin xyz="0 0 -0.018" rpy="0.0 0.0 0.0"/>
+      <parent link="${name}_right_eye_peripheral_link"/>
+      <child link="${name}_right_eye_foveal_link"/>
+    </joint>
+    <link name="${name}_right_eye_foveal_link">
+      <inertial>
+        <xacro:insert_block name="negligible_inertia"/>
+      </inertial>
+      <visual>
+        <origin xyz="0 0 0" rpy="0 0 0"/>
+        <geometry>
+          <sphere radius="0.018"/>
+        </geometry>
+        <material name="KIT/White"/>
+      </visual>
+      <collision>
+        <origin xyz="0 0 0" rpy="0 0 0"/>
+        <geometry>
+          <sphere radius="0.018"/>
         </geometry>
       </collision>
@@ -270,5 +316,5 @@
       </collision>
     </link> -->
-    <joint name="${name}_asus_joint" type="fixed">
+    <!--<joint name="${name}_asus_joint" type="fixed">
       <origin xyz="0 -0.1 0" rpy="1.5707 0.0 0.0"/>
       <parent link="${name}_head_5_link"/>
@@ -292,5 +338,5 @@
         </geometry>
       </collision>
-    </link>
+    </link> !-->
     <xacro:kit_head_transmission name="${name}"/>
     <xacro:kit_head_gazebo name="${name}"/>

Commit message: visualisation and kinematics adjusted a little more

File: kit_head_description/model/kit_head.urdf.xacro (robot description, xacro)
@@ -8,5 +8,5 @@
   <xacro:property name="velocity_scale_factor" value="1.0"/>
   <xacro:macro name="kit_head" params="parent name *origin">
-    <!-- The base of the hand, fixed to its parent. -->
+    <!-- The base of the head, fixed to its parent. -->
     <joint name="${parent}_${name}_base_joint" type="fixed">
       <xacro:insert_block name="origin"/>
@@ -18,12 +18,12 @@
         <xacro:insert_block name="negligible_inertia"/>
       </inertial>
-      <!-- <visual>
-        <origin xyz="0 0 0" rpy="0 0 0"/>
-        <geometry>
-          <cylinder radius="0.03" length="0.15"/>
-        </geometry>
-        <material name="KIT/DarkGrey"/>
-      </visual>
-      <collision>
+       <visual>
+        <origin xyz="0 0 0.05" rpy="0 0 0"/>
+        <geometry>
+          <box size="0.25 0.25 0.1"/>
+        </geometry>
+        <material name="KIT/DarkGrey"/>
+      </visual>
+      <!--<collision>
         <origin xyz="0 0 0" rpy="0 0 0"/>
         <geometry>
@@ -34,5 +34,5 @@
     <!-- neck -->
     <joint name="${name}_neck_pitch_joint" type="revolute">
-      <origin xyz="0 0 0" rpy="${-1*M_PI/2} 0 0"/>
+      <origin xyz="0 0 0.168" rpy="${-1*M_PI/2} 0 0"/>
       <axis xyz="0 0 1"/>
       <limit lower="${-33 * M_PI / 180}" upper="${33 * M_PI / 180}"
@@ -188,6 +188,7 @@
       </collision>
     </link>
+		<!-- -9 mm to go to the upper eye -->
     <joint name="${name}_left_eye_joint" type="revolute">
-      <origin xyz="0 0 0.0465" rpy="${M_PI/2} 0 0"/>
+      <origin xyz="0 -0.009 0.0465" rpy="${M_PI/2} 0 0"/>
       <axis xyz="0 0 1"/>
       <limit lower="${-20 * M_PI / 180}" upper="${20 * M_PI / 180}"
@@ -206,7 +207,7 @@
       </inertial>
       <visual>
-        <origin xyz="0.0 0 0.018" rpy="0 ${M_PI/2} 0"/>
-        <geometry>
-          <sphere radius="0.018"/>
+        <origin xyz="0.0 0 0.0" rpy="0 ${M_PI/2} 0"/>
+        <geometry>
+          <sphere radius="0.009"/>
         </geometry>
         <material name="KIT/White"/>
@@ -215,5 +216,5 @@
         <origin xyz="0.0 0 0" rpy="0 ${M_PI/2} 0"/>
         <geometry>
-          <sphere radius="0.018"/>
+          <sphere radius="0.009"/>
         </geometry>
       </collision>
@@ -231,5 +232,5 @@
         <origin xyz="0 0 0" rpy="0 0 0"/>
         <geometry>
-          <sphere radius="0.018"/>
+          <sphere radius="0.009"/>
         </geometry>
         <material name="KIT/White"/>
@@ -238,10 +239,11 @@
         <origin xyz="0 0 0" rpy="0 0 0"/>
         <geometry>
-          <sphere radius="0.018"/>
-        </geometry>
-      </collision>
-    </link>
+          <sphere radius="0.009"/>
+        </geometry>
+      </collision>
+    </link>
+		<!-- -9 mm to go to the upper eye -->
     <joint name="${name}_right_eye_joint" type="revolute">
-      <origin xyz="0 0 -0.0465" rpy="${M_PI/2} 0 0"/>
+      <origin xyz="0 -0.009 -0.0465" rpy="${M_PI/2} 0 0"/>
       <axis xyz="0 0 1"/>
       <limit lower="${-20 * M_PI / 180}" upper="${20 * M_PI / 180}"
@@ -260,7 +262,7 @@
       </inertial>
       <visual>
-        <origin xyz="0.0 0 0.018" rpy="0 ${M_PI/2} 0"/>
-        <geometry>
-          <sphere radius="0.018"/>
+        <origin xyz="0.0 0 0.0" rpy="0 ${M_PI/2} 0"/>
+        <geometry>
+          <sphere radius="0.009"/>
         </geometry>
         <material name="KIT/White"/>
@@ -269,5 +271,5 @@
         <origin xyz="0.0 0 0" rpy="0 ${M_PI/2} 0"/>
         <geometry>
-          <sphere radius="0.018"/>
+          <sphere radius="0.009"/>
         </geometry>
       </collision>
@@ -285,5 +287,5 @@
         <origin xyz="0 0 0" rpy="0 0 0"/>
         <geometry>
-          <sphere radius="0.018"/>
+          <sphere radius="0.009"/>
         </geometry>
         <material name="KIT/White"/>
@@ -292,5 +294,5 @@
         <origin xyz="0 0 0" rpy="0 0 0"/>
         <geometry>
-          <sphere radius="0.018"/>
+          <sphere radius="0.009"/>
         </geometry>
       </collision>
