Commit message: Fix some mismatches between URDF & Gazebo models
Fix some deprecation warnings.

File: kit_head_description/model/kit_head.gazebo.xacro (robot description, xacro)
@@ -10,37 +10,37 @@
 			<kd>1.0</kd>
 		</gazebo>
-		<gazebo reference="${name}_head_1_link">
-			<!-- selfCollide>true</selfCollide -->
-			<gravity>true</gravity>
-			<mu1>500.0</mu1>
-			<mu2>500.0</mu2>
-			<kp>10000000.0</kp>
-			<kd>1.0</kd>
-		</gazebo>
-		<gazebo reference="${name}_head_2_link">
-			<!-- selfCollide>true</selfCollide -->
-			<gravity>true</gravity>
-			<mu1>500.0</mu1>
-			<mu2>500.0</mu2>
-			<kp>10000000.0</kp>
-			<kd>1.0</kd>
-		</gazebo>
-		<gazebo reference="${name}_head_3_link">
-			<!-- selfCollide>true</selfCollide -->
-			<gravity>true</gravity>
-			<mu1>500.0</mu1>
-			<mu2>500.0</mu2>
-			<kp>10000000.0</kp>
-			<kd>1.0</kd>
-		</gazebo>
-		<gazebo reference="${name}_head_4_link">
-			<!-- selfCollide>true</selfCollide -->
-			<gravity>true</gravity>
-			<mu1>500.0</mu1>
-			<mu2>500.0</mu2>
-			<kp>10000000.0</kp>
-			<kd>1.0</kd>
-		</gazebo>
-		<gazebo reference="${name}_head_5_link">
+		<gazebo reference="${name}_neck_pitch_link">
+			<!-- selfCollide>true</selfCollide -->
+			<gravity>true</gravity>
+			<mu1>500.0</mu1>
+			<mu2>500.0</mu2>
+			<kp>10000000.0</kp>
+			<kd>1.0</kd>
+		</gazebo>
+		<gazebo reference="${name}_neck_roll_link">
+			<!-- selfCollide>true</selfCollide -->
+			<gravity>true</gravity>
+			<mu1>500.0</mu1>
+			<mu2>500.0</mu2>
+			<kp>10000000.0</kp>
+			<kd>1.0</kd>
+		</gazebo>
+		<gazebo reference="${name}_neck_yaw_link">
+			<!-- selfCollide>true</selfCollide -->
+			<gravity>true</gravity>
+			<mu1>500.0</mu1>
+			<mu2>500.0</mu2>
+			<kp>10000000.0</kp>
+			<kd>1.0</kd>
+		</gazebo>
+		<gazebo reference="${name}_neck_tilt_link">
+			<!-- selfCollide>true</selfCollide -->
+			<gravity>true</gravity>
+			<mu1>500.0</mu1>
+			<mu2>500.0</mu2>
+			<kp>10000000.0</kp>
+			<kd>1.0</kd>
+		</gazebo>
+		<gazebo reference="${name}_eyes_tilt_link">
 			<!-- selfCollide>true</selfCollide -->
 			<gravity>true</gravity>

File: kit_head_description/model/kit_head.transmission.xacro (robot description, xacro)
@@ -5,5 +5,5 @@
 			<type>transmission_interface/SimpleTransmission</type>
 			<joint name="${name}_neck_pitch_joint">
-				<hardwareInterface>EffortJointInterface</hardwareInterface>
+        <hardwareInterface>hardware_interface/EffortJointInterface</hardwareInterface>
 			</joint>
 			<actuator name="${name}_neck_pitch_joint_motor">
@@ -14,5 +14,5 @@
 			<type>transmission_interface/SimpleTransmission</type>
 			<joint name="${name}_neck_roll_joint">
-				<hardwareInterface>EffortJointInterface</hardwareInterface>
+        <hardwareInterface>hardware_interface/EffortJointInterface</hardwareInterface>
 			</joint>
 			<actuator name="${name}_neck_roll_joint_motor">
@@ -23,5 +23,5 @@
 			<type>transmission_interface/SimpleTransmission</type>
 			<joint name="${name}_neck_yaw_joint">
-				<hardwareInterface>EffortJointInterface</hardwareInterface>
+        <hardwareInterface>hardware_interface/EffortJointInterface</hardwareInterface>
 			</joint>
 			<actuator name="${name}_neck_yaw_joint_motor">
@@ -29,10 +29,10 @@
 			</actuator>
 		</transmission>
-		<transmission name="${name}_head_tilt_joint_trans">
+		<transmission name="${name}_neck_tilt_joint_trans">
 			<type>transmission_interface/SimpleTransmission</type>
-			<joint name="${name}_head_tilt_joint">
-				<hardwareInterface>EffortJointInterface</hardwareInterface>
+			<joint name="${name}_neck_tilt_joint">
+        <hardwareInterface>hardware_interface/EffortJointInterface</hardwareInterface>
 			</joint>
-			<actuator name="${name}_head_tilt_joint_motor">
+			<actuator name="${name}_neck_tilt_joint_motor">
 				<mechanicalReduction>1.0</mechanicalReduction>
 			</actuator>
@@ -41,5 +41,5 @@
 			<type>transmission_interface/SimpleTransmission</type>
 			<joint name="${name}_eyes_tilt_joint">
-				<hardwareInterface>EffortJointInterface</hardwareInterface>
+        <hardwareInterface>hardware_interface/EffortJointInterface</hardwareInterface>
 			</joint>
 			<actuator name="${name}_eyes_tilt_joint_motor">
@@ -50,5 +50,5 @@
 			<type>transmission_interface/SimpleTransmission</type>
 			<joint name="${name}_left_eye_joint">
-				<hardwareInterface>EffortJointInterface</hardwareInterface>
+        <hardwareInterface>hardware_interface/EffortJointInterface</hardwareInterface>
 			</joint>
 			<actuator name="${name}_left_eye_joint_motor">
@@ -59,5 +59,5 @@
 			<type>transmission_interface/SimpleTransmission</type>
 			<joint name="${name}_right_eye_joint">
-				<hardwareInterface>EffortJointInterface</hardwareInterface>
+        <hardwareInterface>hardware_interface/EffortJointInterface</hardwareInterface>
 			</joint>
 			<actuator name="${name}_right_eye_joint_motor">

Commit message: some changes, forgot what about

File: kit_head_description/model/kit_head.gazebo.xacro (robot description, xacro)
@@ -10,37 +10,37 @@
 			<kd>1.0</kd>
 		</gazebo>
-		<gazebo reference="${name}_neck_pitch_link">
-			<!-- selfCollide>true</selfCollide -->
-			<gravity>true</gravity>
-			<mu1>500.0</mu1>
-			<mu2>500.0</mu2>
-			<kp>10000000.0</kp>
-			<kd>1.0</kd>
-		</gazebo>
-		<gazebo reference="${name}_neck_roll_link">
-			<!-- selfCollide>true</selfCollide -->
-			<gravity>true</gravity>
-			<mu1>500.0</mu1>
-			<mu2>500.0</mu2>
-			<kp>10000000.0</kp>
-			<kd>1.0</kd>
-		</gazebo>
-		<gazebo reference="${name}_neck_yaw_link">
-			<!-- selfCollide>true</selfCollide -->
-			<gravity>true</gravity>
-			<mu1>500.0</mu1>
-			<mu2>500.0</mu2>
-			<kp>10000000.0</kp>
-			<kd>1.0</kd>
-		</gazebo>
-		<gazebo reference="${name}_neck_tilt_link">
-			<!-- selfCollide>true</selfCollide -->
-			<gravity>true</gravity>
-			<mu1>500.0</mu1>
-			<mu2>500.0</mu2>
-			<kp>10000000.0</kp>
-			<kd>1.0</kd>
-		</gazebo>
-		<gazebo reference="${name}_eyes_tilt_link">
+		<gazebo reference="${name}_head_1_link">
+			<!-- selfCollide>true</selfCollide -->
+			<gravity>true</gravity>
+			<mu1>500.0</mu1>
+			<mu2>500.0</mu2>
+			<kp>10000000.0</kp>
+			<kd>1.0</kd>
+		</gazebo>
+		<gazebo reference="${name}_head_2_link">
+			<!-- selfCollide>true</selfCollide -->
+			<gravity>true</gravity>
+			<mu1>500.0</mu1>
+			<mu2>500.0</mu2>
+			<kp>10000000.0</kp>
+			<kd>1.0</kd>
+		</gazebo>
+		<gazebo reference="${name}_head_3_link">
+			<!-- selfCollide>true</selfCollide -->
+			<gravity>true</gravity>
+			<mu1>500.0</mu1>
+			<mu2>500.0</mu2>
+			<kp>10000000.0</kp>
+			<kd>1.0</kd>
+		</gazebo>
+		<gazebo reference="${name}_head_4_link">
+			<!-- selfCollide>true</selfCollide -->
+			<gravity>true</gravity>
+			<mu1>500.0</mu1>
+			<mu2>500.0</mu2>
+			<kp>10000000.0</kp>
+			<kd>1.0</kd>
+		</gazebo>
+		<gazebo reference="${name}_head_5_link">
 			<!-- selfCollide>true</selfCollide -->
 			<gravity>true</gravity>

File: kit_head_description/model/kit_head.transmission.xacro (robot description, xacro)
@@ -5,5 +5,5 @@
 			<type>transmission_interface/SimpleTransmission</type>
 			<joint name="${name}_neck_pitch_joint">
-        <hardwareInterface>hardware_interface/EffortJointInterface</hardwareInterface>
+				<hardwareInterface>EffortJointInterface</hardwareInterface>
 			</joint>
 			<actuator name="${name}_neck_pitch_joint_motor">
@@ -14,5 +14,5 @@
 			<type>transmission_interface/SimpleTransmission</type>
 			<joint name="${name}_neck_roll_joint">
-        <hardwareInterface>hardware_interface/EffortJointInterface</hardwareInterface>
+				<hardwareInterface>EffortJointInterface</hardwareInterface>
 			</joint>
 			<actuator name="${name}_neck_roll_joint_motor">
@@ -23,5 +23,5 @@
 			<type>transmission_interface/SimpleTransmission</type>
 			<joint name="${name}_neck_yaw_joint">
-        <hardwareInterface>hardware_interface/EffortJointInterface</hardwareInterface>
+				<hardwareInterface>EffortJointInterface</hardwareInterface>
 			</joint>
 			<actuator name="${name}_neck_yaw_joint_motor">
@@ -29,10 +29,10 @@
 			</actuator>
 		</transmission>
-		<transmission name="${name}_neck_tilt_joint_trans">
+		<transmission name="${name}_head_tilt_joint_trans">
 			<type>transmission_interface/SimpleTransmission</type>
-			<joint name="${name}_neck_tilt_joint">
-        <hardwareInterface>hardware_interface/EffortJointInterface</hardwareInterface>
+			<joint name="${name}_head_tilt_joint">
+				<hardwareInterface>EffortJointInterface</hardwareInterface>
 			</joint>
-			<actuator name="${name}_neck_tilt_joint_motor">
+			<actuator name="${name}_head_tilt_joint_motor">
 				<mechanicalReduction>1.0</mechanicalReduction>
 			</actuator>
@@ -41,5 +41,5 @@
 			<type>transmission_interface/SimpleTransmission</type>
 			<joint name="${name}_eyes_tilt_joint">
-        <hardwareInterface>hardware_interface/EffortJointInterface</hardwareInterface>
+				<hardwareInterface>EffortJointInterface</hardwareInterface>
 			</joint>
 			<actuator name="${name}_eyes_tilt_joint_motor">
@@ -50,5 +50,5 @@
 			<type>transmission_interface/SimpleTransmission</type>
 			<joint name="${name}_left_eye_joint">
-        <hardwareInterface>hardware_interface/EffortJointInterface</hardwareInterface>
+				<hardwareInterface>EffortJointInterface</hardwareInterface>
 			</joint>
 			<actuator name="${name}_left_eye_joint_motor">
@@ -59,5 +59,5 @@
 			<type>transmission_interface/SimpleTransmission</type>
 			<joint name="${name}_right_eye_joint">
-        <hardwareInterface>hardware_interface/EffortJointInterface</hardwareInterface>
+				<hardwareInterface>EffortJointInterface</hardwareInterface>
 			</joint>
 			<actuator name="${name}_right_eye_joint_motor">

File: kit_head_description/model/kit_head.urdf.xacro (robot description, xacro)
@@ -8,5 +8,5 @@
   <xacro:property name="velocity_scale_factor" value="1.0"/>
   <xacro:macro name="kit_head" params="parent name *origin">
-    <!-- The base of the head, fixed to its parent. -->
+    <!-- The base of the hand, fixed to its parent. -->
     <joint name="${parent}_${name}_base_joint" type="fixed">
       <xacro:insert_block name="origin"/>
@@ -18,12 +18,12 @@
         <xacro:insert_block name="negligible_inertia"/>
       </inertial>
-       <visual>
-        <origin xyz="0 0 0.05" rpy="0 0 0"/>
-        <geometry>
-          <box size="0.25 0.25 0.1"/>
-        </geometry>
-        <material name="KIT/DarkGrey"/>
-      </visual>
-      <!--<collision>
+      <!-- <visual>
+        <origin xyz="0 0 0" rpy="0 0 0"/>
+        <geometry>
+          <cylinder radius="0.03" length="0.15"/>
+        </geometry>
+        <material name="KIT/DarkGrey"/>
+      </visual>
+      <collision>
         <origin xyz="0 0 0" rpy="0 0 0"/>
         <geometry>
@@ -34,5 +34,5 @@
     <!-- neck -->
     <joint name="${name}_neck_pitch_joint" type="revolute">
-      <origin xyz="0 0 0.168" rpy="${-1*M_PI/2} 0 0"/>
+      <origin xyz="0 0 0" rpy="${-1*M_PI/2} 0 0"/>
       <axis xyz="0 0 1"/>
       <limit lower="${-33 * M_PI / 180}" upper="${33 * M_PI / 180}"
@@ -44,7 +44,7 @@
       <dynamics friction="1.0" damping="1.0"/>
       <parent link="${name}_base_link"/>
-      <child link="${name}_neck_pitch_link"/>
-    </joint>
-    <link name="${name}_neck_pitch_link">
+      <child link="${name}_head_1_link"/>
+    </joint>
+    <link name="${name}_head_1_link">
       <inertial>
         <xacro:insert_block name="negligible_inertia"/>
@@ -74,8 +74,8 @@
                          k_velocity="30"/>
       <dynamics friction="1.0" damping="1.0"/>
-      <parent link="${name}_neck_pitch_link"/>
-      <child link="${name}_neck_roll_link"/>
-    </joint>
-    <link name="${name}_neck_roll_link">
+      <parent link="${name}_head_1_link"/>
+      <child link="${name}_head_2_link"/>
+    </joint>
+    <link name="${name}_head_2_link">
       <inertial>
         <xacro:insert_block name="negligible_inertia"/>
@@ -105,27 +105,27 @@
                          k_velocity="30"/>
       <dynamics friction="1.0" damping="1.0"/>
-      <parent link="${name}_neck_roll_link"/>
-      <child link="${name}_neck_yaw_link"/>
-    </joint>
-    <link name="${name}_neck_yaw_link">
-      <inertial>
-        <xacro:insert_block name="negligible_inertia"/>
-      </inertial>
-      <visual>
-        <origin xyz="0 0 0" rpy="0 0 0"/>
-        <geometry>
-          <cylinder radius="0.03" length="0.15"/>
-        </geometry>
-        <material name="KIT/DarkGrey"/>
-      </visual>
-      <collision>
-        <origin xyz="0 0 0" rpy="0 0 0"/>
-        <geometry>
-          <cylinder radius="0.03" length="0.15"/>
-        </geometry>
-      </collision>
-    </link>
-    <joint name="${name}_neck_tilt_joint" type="revolute">
-      <origin xyz="0 0 -0.122" rpy="${M_PI/2} 0 0"/>
+      <parent link="${name}_head_2_link"/>
+      <child link="${name}_head_3_link"/>
+    </joint>
+    <link name="${name}_head_3_link">
+      <inertial>
+        <xacro:insert_block name="negligible_inertia"/>
+      </inertial>
+      <visual>
+        <origin xyz="0 0 0" rpy="0 0 0"/>
+        <geometry>
+          <cylinder radius="0.03" length="0.15"/>
+        </geometry>
+        <material name="KIT/DarkGrey"/>
+      </visual>
+      <collision>
+        <origin xyz="0 0 0" rpy="0 0 0"/>
+        <geometry>
+          <cylinder radius="0.03" length="0.15"/>
+        </geometry>
+      </collision>
+    </link>
+    <joint name="${name}_head_tilt_joint" type="revolute">
+      <origin xyz="0 0 -0.1745" rpy="${M_PI/2} 0 0"/>
       <axis xyz="0 0 1"/>
       <limit lower="${-40 * M_PI / 180}" upper="${40 * M_PI / 180}"
@@ -136,8 +136,8 @@
                          k_velocity="30"/>
       <dynamics friction="1.0" damping="1.0"/>
-      <parent link="${name}_neck_yaw_link"/>
-      <child link="${name}_neck_tilt_link"/>
-    </joint>
-    <link name="${name}_neck_tilt_link">
+      <parent link="${name}_head_3_link"/>
+      <child link="${name}_head_4_link"/>
+    </joint>
+    <link name="${name}_head_4_link">
       <inertial>
         <xacro:insert_block name="negligible_inertia"/>
@@ -158,5 +158,5 @@
     </link>
     <joint name="${name}_eyes_tilt_joint" type="revolute">
-      <origin xyz="0.1 -0.0525 0.0" rpy="0 0 0"/>
+      <origin xyz="0.1 0 0" rpy="0 0 0"/>
       <axis xyz="0 0 1"/>
       <limit lower="${-20 * M_PI / 180}" upper="${20 * M_PI / 180}"
@@ -167,8 +167,8 @@
                          k_velocity="30"/>
       <dynamics friction="1.0" damping="1.0"/>
-      <parent link="${name}_neck_tilt_link"/>
-      <child link="${name}_eyes_tilt_link"/>
-    </joint>
-    <link name="${name}_eyes_tilt_link">
+      <parent link="${name}_head_4_link"/>
+      <child link="${name}_head_5_link"/>
+    </joint>
+    <link name="${name}_head_5_link">
       <inertial>
         <xacro:insert_block name="negligible_inertia"/>
@@ -188,7 +188,6 @@
       </collision>
     </link>
-		<!-- -9 mm to go to the upper eye -->
     <joint name="${name}_left_eye_joint" type="revolute">
-      <origin xyz="0 -0.009 0.0465" rpy="${M_PI/2} 0 0"/>
+      <origin xyz="0 0 0.0465" rpy="${M_PI/2} 0 0"/>
       <axis xyz="0 0 1"/>
       <limit lower="${-20 * M_PI / 180}" upper="${20 * M_PI / 180}"
@@ -199,51 +198,27 @@
                          k_velocity="30"/>
       <dynamics friction="1.0" damping="1.0"/>
-      <parent link="${name}_eyes_tilt_link"/>
-      <child link="${name}_left_eye_peripheral_link"/>
-    </joint>
-    <link name="${name}_left_eye_peripheral_link">
-      <inertial>
-        <xacro:insert_block name="negligible_inertia"/>
-      </inertial>
-      <visual>
-        <origin xyz="0.0 0 0.0" rpy="0 ${M_PI/2} 0"/>
-        <geometry>
-          <sphere radius="0.009"/>
+      <parent link="${name}_head_5_link"/>
+      <child link="${name}_left_eye_link"/>
+    </joint>
+    <link name="${name}_left_eye_link">
+      <inertial>
+        <xacro:insert_block name="negligible_inertia"/>
+      </inertial>
+      <visual>
+        <origin xyz="0.02 0 0" rpy="0 ${M_PI/2} 0"/>
+        <geometry>
+          <cylinder radius="0.03" length="0.02"/>
         </geometry>
         <material name="KIT/White"/>
       </visual>
       <collision>
-        <origin xyz="0.0 0 0" rpy="0 ${M_PI/2} 0"/>
-        <geometry>
-          <sphere radius="0.009"/>
-        </geometry>
-      </collision>
-    </link>
-    <joint name="${name}_left_eye_foveal_joint" type="fixed">
-      <origin xyz="0 0 -0.018" rpy="0.0 0.0 0.0"/>
-      <parent link="${name}_left_eye_peripheral_link"/>
-      <child link="${name}_left_eye_foveal_link"/>
-    </joint>
-    <link name="${name}_left_eye_foveal_link">
-      <inertial>
-        <xacro:insert_block name="negligible_inertia"/>
-      </inertial>
-      <visual>
-        <origin xyz="0 0 0" rpy="0 0 0"/>
-        <geometry>
-          <sphere radius="0.009"/>
-        </geometry>
-        <material name="KIT/White"/>
-      </visual>
-      <collision>
-        <origin xyz="0 0 0" rpy="0 0 0"/>
-        <geometry>
-          <sphere radius="0.009"/>
-        </geometry>
-      </collision>
-    </link>
-		<!-- -9 mm to go to the upper eye -->
+        <origin xyz="0.02 0 0" rpy="0 ${M_PI/2} 0"/>
+        <geometry>
+          <cylinder radius="0.03" length="0.02"/>
+        </geometry>
+      </collision>
+    </link>
     <joint name="${name}_right_eye_joint" type="revolute">
-      <origin xyz="0 -0.009 -0.0465" rpy="${M_PI/2} 0 0"/>
+      <origin xyz="0 0 -0.0465" rpy="${M_PI/2} 0 0"/>
       <axis xyz="0 0 1"/>
       <limit lower="${-20 * M_PI / 180}" upper="${20 * M_PI / 180}"
@@ -254,45 +229,22 @@
                          k_velocity="30"/>
       <dynamics friction="1.0" damping="1.0"/>
-      <parent link="${name}_eyes_tilt_link"/>
-      <child link="${name}_right_eye_peripheral_link"/>
-    </joint>
-    <link name="${name}_right_eye_peripheral_link">
-      <inertial>
-        <xacro:insert_block name="negligible_inertia"/>
-      </inertial>
-      <visual>
-        <origin xyz="0.0 0 0.0" rpy="0 ${M_PI/2} 0"/>
-        <geometry>
-          <sphere radius="0.009"/>
+      <parent link="${name}_head_5_link"/>
+      <child link="${name}_right_eye_link"/>
+    </joint>
+    <link name="${name}_right_eye_link">
+      <inertial>
+        <xacro:insert_block name="negligible_inertia"/>
+      </inertial>
+      <visual>
+        <origin xyz="0.02 0 0" rpy="0 ${M_PI/2} 0"/>
+        <geometry>
+          <cylinder radius="0.03" length="0.02"/>
         </geometry>
         <material name="KIT/White"/>
       </visual>
       <collision>
-        <origin xyz="0.0 0 0" rpy="0 ${M_PI/2} 0"/>
-        <geometry>
-          <sphere radius="0.009"/>
-        </geometry>
-      </collision>
-    </link>
-    <joint name="${name}_right_eye_foveal_joint" type="fixed">
-      <origin xyz="0 0 -0.018" rpy="0.0 0.0 0.0"/>
-      <parent link="${name}_right_eye_peripheral_link"/>
-      <child link="${name}_right_eye_foveal_link"/>
-    </joint>
-    <link name="${name}_right_eye_foveal_link">
-      <inertial>
-        <xacro:insert_block name="negligible_inertia"/>
-      </inertial>
-      <visual>
-        <origin xyz="0 0 0" rpy="0 0 0"/>
-        <geometry>
-          <sphere radius="0.009"/>
-        </geometry>
-        <material name="KIT/White"/>
-      </visual>
-      <collision>
-        <origin xyz="0 0 0" rpy="0 0 0"/>
-        <geometry>
-          <sphere radius="0.009"/>
+        <origin xyz="0.02 0 0" rpy="0 ${M_PI/2} 0"/>
+        <geometry>
+          <cylinder radius="0.03" length="0.02"/>
         </geometry>
       </collision>
@@ -318,5 +270,5 @@
       </collision>
     </link> -->
-    <!--<joint name="${name}_asus_joint" type="fixed">
+    <joint name="${name}_asus_joint" type="fixed">
       <origin xyz="0 -0.1 0" rpy="1.5707 0.0 0.0"/>
       <parent link="${name}_head_5_link"/>
@@ -340,5 +292,5 @@
         </geometry>
       </collision>
-    </link> !-->
+    </link>
     <xacro:kit_head_transmission name="${name}"/>
     <xacro:kit_head_gazebo name="${name}"/>
